File: pcb/cheating-calc.kicad_pcb (KiCad board)
At the start: 2 copper layers, 72 x 22 mm, 8 parts, among them J1 Conn_01x04, Q1 MMBF170, Q2 MMBF170, U1 MOUDLE-SEEEDUINO-XIAO-ESP32C3

Commit message: Update PCB files and documentation from Ti-84-yeet
- Replaced PCB files with updated versions
- Updated README with proper documentation
- Added Chromalock.pdf reference
- Marked GPT display bug as fixed
- Updated author credits
Other:
- board text added: "TI-84 Hacks AndyPandy 2025"
- board text removed: "TI-32 v0.1 ChromaLock 2024"
